File: Power-supply.kicad_sch (KiCad schematic)
At the start: 27 parts, among them J10 USB_C_Receptacle_USB2.0_16P, J11 Conn_01x02, J12 EXT_PWR, J13 Conn_02x03_Odd_Even, Q1 MMBT2222A, U2 TL431DBZ, U3 SPX3819M5-L-3-3, U4 AMS1117-5.0

Commit message: SMD part number assigned, relocate MCU sch to hierarcical sheet
Parts:
- C17: JLCPCB Part # (none) -> C14858
- C18, C23, C25: JLCPCB Part # (none) -> C14663
- C20, C27: JLCPCB Part # (none) -> C440198
- C22: JLCPCB Part # (none) -> C28323
- C24: JLCPCB Part # (none) -> C377773
- C26: JLCPCB Part # (none) -> C57112
- C28: JLCPCB Part # (none) -> C45783
- D4: value LED -> GREEN; JLCPCB Part # (none) -> C2297
- J10: JLCPCB Part # (none) -> C2988369
- J11, J12, J13: now left out of the parts list
- Q1: JLCPCB Part # (none) -> C82460
- R1: JLCPCB Part # (none) -> C22828
- R10, R11: JLCPCB Part # (none) -> C23186
- R12: JLCPCB Part # (none) -> C23192
- R2: JLCPCB Part # (none) -> C227439
- R3: JLCPCB Part # (none) -> C227486
- U2: JLCPCB Part # (none) -> C23892
- U3: JLCPCB Part # (none) -> C5370980
- U4: JLCPCB Part # (none) -> C6187
