File: STM32G474RE.kicad_sch (KiCad schematic)
At the start: 37 parts, among them J1 Conn_01x02, J16 Conn_01x03, J17 Conn_02x05_Odd_Even, J2 ST-LINK, J8 Conn_01x02, SW1 SW_Push, SW2 SW_Push, U1 STM32G474RETx, Y1 24MHz, Y2 32.768KHz

Commit message: no changes
Changed lines of the file:
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@@
+		)
+	)
+	(bus
+		(pts
+			(xy 59.69 180.34) (xy 68.58 180.34)
+		)
+		(stroke
+			(width 0)
+			(type default)
 		)
 	)
@@
 	(wire
 		(pts
+			(xy 59.69 193.04) (xy 68.58 193.04)
+		)
+		(stroke
+			(width 0)
+			(type default)
+		)
+	)
+	(wire
+		(pts
+			(xy 59.69 187.96) (xy 68.58 187.96)
+		)
+		(stroke
+			(width 0)
+			(type default)
+		)
+	)
+	(wire
+		(pts
 			(xy 31.75 97.79) (xy 35.56 97.79)
 		)
@@
 	(wire
 		(pts
+			(xy 59.69 190.5) (xy 68.58 190.5)
+		)
+		(stroke
+			(width 0)
+			(type default)
+		)
+	)
+	(wire
+		(pts
 			(xy 90.17 55.88) (xy 92.71 55.88)
 		)
@@
 	(wire
 		(pts
+			(xy 59.69 185.42) (xy 68.58 185.42)
+		)
+		(stroke
+			(width 0)
+			(type default)
+		)
+	)
+	(wire
+		(pts
 			(xy 156.21 59.69) (xy 156.21 63.5)
 		)
@@
 		)
 	)
+	(bus
+		(pts
+			(xy 59.69 177.8) (xy 68.58 177.8)
+		)
+		(stroke
+			(width 0)
+			(type default)
+		)
+	)
 	(wire
 		(pts
@@
 		(pts
 			(xy 157.48 104.14) (xy 157.48 106.68)
+		)
+		(stroke
+			(width 0)
+			(type default)
+		)
+	)
+	(bus
+		(pts
+			(xy 59.69 182.88) (xy 68.58 182.88)
 		)
 		(stroke
@@
 		)
 	)
+	(hierarchical_label "NRST"
+		(shape input)
+		(at 68.58 190.5 0)
+		(fields_autoplaced yes)
+		(effects
+			(font
+				(size 1.27 1.27)
+			)
+			(justify left)
+		)
+	)
+	(hierarchical_label "PA[0..15]"
+		(shape bidirectional)
+		(at 68.58 177.8 0)
+		(fields_autoplaced yes)
+		(effects
+			(font
+				(size 1.27 1.27)
+			)
+			(justify left)
+		)
+	)
+	(hierarchical_label "BOOT"
+		(shape input)
+		(at 68.58 187.96 0)
+		(fields_autoplaced yes)
+		(effects
+			(font
+				(size 1.27 1.27)
+			)
+			(justify left)
+		)
+	)
+	(hierarchical_label "PC[0..15]"
+		(shape bidirectional)
+		(at 68.58 182.88 0)
+		(fields_autoplaced yes)
+		(effects
+			(font
+				(size 1.27 1.27)
+			)
+			(justify left)
+		)
+	)
+	(hierarchical_label "PB[0..15]"
+		(shape bidirectional)
+		(at 68.58 180.34 0)
+		(fields_autoplaced yes)
+		(effects
+			(font
+				(size 1.27 1.27)
+			)
+			(justify left)
+		)
+	)
+	(hierarchical_label "VBAT"
+		(shape input)
+		(at 68.58 193.04 0)
+		(fields_autoplaced yes)
+		(effects
+			(font
+				(size 1.27 1.27)
+			)
+			(justify left)
+		)
+	)
 	(hierarchical_label "BOOT"
 		(shape input)
@@
 		(fields_autoplaced yes)
 		(effects
+			(font
+				(size 1.27 1.27)
+			)
+			(justify left)
+		)
+	)
+	(hierarchical_label "PD2"
+		(shape bidirectional)
+		(at 68.58 185.42 0)
+		(fields_autoplaced yes)
+		(effects
